File: F9P_Carrier_Board.sch (EAGLE design)
At the start: 79 parts, among them J4 U.FL, J5 QWIIC_RIGHT_ANGLE, J6 MICROMOD-2222-C, J8 JTAG, U1 U-BLOX_ZED-F9P, U5 AP7361C-33

Commit message: Fixes nets on the ZED-F9P, fixes silk, removes excessive GND vias, adds SMA connector for PPS
* Fixes 12 pin header
* Fixes jumper labels in schematic
* Fixes RX/TX lines, and SDO/SDI lines
* Adds version number
Parts:
- added D12, D5: 3A/10V/280mV, SparkFun-DiscreteSemi:DIODE-SCHOTTKY-BAT60A
- added E1: ANTENNA-SMA-GROUNDEDEDGE_SMA, SparkFun-RF:ANTENNA-SMA-GROUNDEDEDGE_SMA
- J10: device SparkFun-Connectors:CONN_121X12_NO_SILK_KIT -> SparkFun-Connectors:CONN_12NO_SILK
- J4: device SparkFun-RF:ANTENNA-GROUNDEDEDGE_SMA_SMD -> SparkFun-RF:ANTENNA-SMA-GROUNDEDEDGE_RPSMA_SMD
- renumbered JP5 to SPI
Connections:
- new net V_FUSE: BYP.1, D12.C, D5.C, F2.1
- new net V_USB_2: D12.A, D4.5, J10.6, J3.VBUS
- net !SAFEBOOT!: now also R11B.2; no longer R11C.2
- net !ZED_RESET!: now also R11C.2; no longer R11B.2
- net GND: now also E1.GND
- net INT: now also J6.D1/CAM_TRIG, R11A.2; no longer J6.G0/BUS0, R11D.2
- net PPS: now also E1.SIGNAL
- net RXI/SDI: now also J6.SPI_SDO, R12C.2; no longer J6.SPI_SDI, R12B.2
- net RXI2: now also J6.TX2; no longer J6.RX2
- net SCL/CLK: now also R12A.2; no longer R12D.2
- net SDA/!CS!: now also R12B.2; no longer R12C.2
- net TXO/SDO: now also J6.SPI_SDI, R12D.2; no longer J6.SPI_SDO, R12A.2
- net TXO2: now also J6.RX2; no longer J6.TX2
- net TX_READY: now also J6.D0, R11D.2; no longer J6.G1/BUS1, R11A.2
- net V_USB: now also D5.A; no longer BYP.1, D4.5, F2.1, J10.6, J3.VBUS
Other:
- note added: "v01"
- note removed: "v10"
- moved on the sheet: BYP, C8, D2, D3, F2, FB1, R17

Commit message: Fixes silk, updates schematic with better labels and descriptions
Other:
- note added: "DNP"
- note added: "GPS and PPS Antenna"
- note removed: "Antenna"
Changed lines of the file:
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@@
 Processor Board</text>
 <text x="424.18" y="7.62" size="2.54" layer="94" font="vector" align="center">v01</text>
-<text x="203.2" y="208.28" size="2.54" layer="94" font="vector" align="center">Antenna</text>
+<text x="203.454" y="210.312" size="2.54" layer="94" font="vector" align="center">GPS and PPS Antenna</text>
 <wire x1="109.22" y1="78.74" x2="0" y2="78.74" width="0.2032" layer="97" style="longdash"/>
 <text x="332.74" y="208.28" size="2.54" layer="94" font="vector" align="center">GPS Module
@@
 <text x="183.134" y="146.05" size="1.27" layer="97" font="vector">Dielectric thickness: 1.46mm</text>
 <text x="183.134" y="153.67" size="1.524" layer="97" font="vector" ratio="15">Co-planar Calculation:</text>
+<text x="229.362" y="194.564" size="2.032" layer="97" font="vector">DNP</text>
+<wire x1="223.52" y1="195.58" x2="228.6" y2="195.58" width="0.2032" layer="97" style="dashdot"/>
 </plain>
 <instances>

Commit message: Removes "INT" trace to MicroMod connector
Connections:
- net INT: no longer J6.D1/CAM_TRIG
Changed lines of the file:
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@@
 <pinref part="R11" gate="A" pin="2"/>
-</segment>
-<segment>
-<pinref part="J6" gate="J1" pin="D1/CAM_TRIG"/>
-<wire x1="106.68" y1="167.64" x2="109.22" y2="167.64" width="0.1524" layer="91"/>
-<label x="109.22" y="167.64" size="1.27" layer="95" xref="yes"/>
 </segment>
 </net>
